File: Low Noise PS Bottom SMD.brd (EAGLE design)
At the start: 228.6 x 101.6 mm, 62 parts, among them IC1 MAX6350SO08, IC2 OP27, IC3 LT1677, IC4 LT1677, IC5 MC79M12CDTG, IC6 MC78M12BDTG, Q1 MMBT2907AMMBTA56SOT23, Q2 MMBT5550SOT23, Q3 PMBF170, Q4 BSH201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

Commit message: Intermediate version
More work is still required
Parts:
- added R17, R18: 10k, rcl:R1206
- moved R7 299.5 mm to (417.8, -80.6)
- moved C25 236.6 mm to (341.0, -22.2), turned to 90 degrees
- moved Q4 235.2 mm to (329.3, -32.0), turned to 180 degrees
- moved C16 234.6 mm to (339.7, -26.0), turned to 180 degrees
- moved R14 230.2 mm to (338.5, -22.2), turned to 270 degrees
- moved R15 228.1 mm to (335.3, -28.6), turned to 180 degrees
- moved R13 224.5 mm to (328.0, -27.2), turned to 90 degrees
- moved C13 222.3 mm to (339.1, -29.8), turned to 90 degrees
- moved Q2 219.5 mm to (334.8, -34.0), turned to 270 degrees
- moved R16 219.1 mm to (330.5, -27.2), turned to 90 degrees
- moved R8 206.8 mm to (330.2, -16.3), turned to 90 degrees
- moved IC4 205.2 mm to (334.8, -23.1)
- moved C12 204.7 mm to (332.9, -16.3), turned to 270 degrees
- moved C19 198.2 mm to (330.4, -21.9), turned to 90 degrees
- moved R4 197.4 mm to (336.6, -14.8), turned to 180 degrees
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Connections:
- net N$22 renamed -12V
- net N$24 renamed +12V
- new net N$12: Q4.1, R16.1, R17.1
- new net N$25: Q3.1, R11.1, R18.1
- net N$28: now also R17.2; no longer Q4.1, R16.1
- net N$35: now also R18.2; no longer Q3.1, R11.1
Routing:
- net N$23: track 0.00 -> 19.8 mm
- net N$28: track 0.00 -> 13.1 mm
- net AGND: track 0.00 -> 8.57 mm, vias 0 -> 2
- net N$35: track 0.00 -> 7.84 mm
- net N$12: track 0.00 -> 6.07 mm
- net N$21: track 0.00 -> 5.82 mm
- net N$10: track 0.00 -> 5.17 mm
- net N$20: track 0.00 -> 4.37 mm
- net N$33: track 0.00 -> 3.39 mm
- net N$11: track 0.00 -> 3.16 mm
- net N$25: track 0.00 -> 3.10 mm
- net N$17: track 0.00 -> 3.10 mm
- net N$18: track 0.00 -> 2.99 mm
- net N$13: track 0.00 -> 2.77 mm
- net N$34: track 0.00 -> 2.74 mm
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