File: Low Noise PS Bottom SMD.sch (EAGLE design)
At the start: 62 parts, among them IC1 MAX6350SO08, IC2 OP27, IC3 LT1677, IC4 LT1677, IC5 MC79M12CDTG, IC6 MC78M12BDTG, Q1 MMBT2907AMMBTA56SOT23, Q2 MMBT5550SOT23, Q3 PMBF170, Q4 BSH201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

Commit message: Intermediate version
More work is still required
Parts:
- added R17, R18: 10k, rcl:R-US_R1206
Connections:
- net N$22 renamed -12V
- net N$24 renamed +12V
- new net N$12: Q4.G, R16.1, R17.1
- new net N$25: Q3.G, R11.1, R18.1
- net N$28: now also R17.2; no longer Q4.G, R16.1
- net N$35: now also R18.2; no longer Q3.G, R11.1
Other:
- moved on the sheet: C25, R14
Changed lines of the file:
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@@
 <part name="AGND21" library="supply1" deviceset="AGND" device=""/>
 <part name="AGND22" library="supply1" deviceset="AGND" device=""/>
+<part name="R17" library="rcl" deviceset="R-US_" device="R1206" value="10k"/>
+<part name="R18" library="rcl" deviceset="R-US_" device="R1206" value="10k"/>
 </parts>
 <sheets>
@@
 <instance part="R13" gate="G$1" x="368.3" y="22.86" rot="R90"/>
 <instance part="C16" gate="G$1" x="335.28" y="35.56" rot="R180"/>
-<instance part="C25" gate="G$1" x="342.9" y="30.48" rot="R180"/>
-<instance part="R14" gate="G$1" x="330.2" y="30.48" rot="R180"/>
+<instance part="C25" gate="G$1" x="335.28" y="30.48" rot="R180"/>
+<instance part="R14" gate="G$1" x="322.58" y="30.48" rot="R180"/>
 <instance part="R15" gate="G$1" x="335.28" y="12.7" rot="R180"/>
 <instance part="R16" gate="G$1" x="358.14" y="20.32" rot="R90"/>
 <instance part="AGND21" gate="VR1" x="375.92" y="25.4"/>
 <instance part="AGND22" gate="VR1" x="363.22" y="22.86"/>
+<instance part="R17" gate="G$1" x="350.52" y="12.7" rot="R180"/>
+<instance part="R18" gate="G$1" x="355.6" y="76.2" rot="R180"/>
 </instances>
 <busses>
@@
 </segment>
 </net>
-<net name="N$22" class="0">
+<net name="-12V" class="0">
 <segment>
 <pinref part="IC5" gate="G$1" pin="VO"/>
@@
 </segment>
 </net>
-<net name="N$24" class="0">
+<net name="+12V" class="0">
 <segment>
 <pinref part="C23" gate="G$1" pin="P$2"/>
@@
 <segment>
 <pinref part="R10" gate="G$1" pin="1"/>
-<pinref part="R11" gate="G$1" pin="1"/>
-<wire x1="347.98" y1="76.2" x2="353.06" y2="76.2" width="0.1524" layer="91"/>
-<pinref part="Q3" gate="G$1" pin="G"/>
-<wire x1="353.06" y1="76.2" x2="360.68" y2="76.2" width="0.1524" layer="91"/>
-<wire x1="360.68" y1="76.2" x2="360.68" y2="71.12" width="0.1524" layer="91"/>
-<wire x1="365.76" y1="76.2" x2="360.68" y2="76.2" width="0.1524" layer="91"/>
+<wire x1="347.98" y1="76.2" x2="350.52" y2="76.2" width="0.1524" layer="91"/>
 <pinref part="C14" gate="G$1" pin="P$1"/>
-<wire x1="345.44" y1="58.42" x2="353.06" y2="58.42" width="0.1524" layer="91"/>
-<wire x1="353.06" y1="58.42" x2="353.06" y2="76.2" width="0.1524" layer="91"/>
+<wire x1="345.44" y1="58.42" x2="350.52" y2="58.42" width="0.1524" layer="91"/>
+<wire x1="350.52" y1="58.42" x2="350.52" y2="76.2" width="0.1524" layer="91"/>
 <pinref part="C15" gate="G$1" pin="P$1"/>
-<wire x1="335.28" y1="53.34" x2="353.06" y2="53.34" width="0.1524" layer="91"/>
-<wire x1="353.06" y1="53.34" x2="353.06" y2="58.42" width="0.1524" layer="91"/>
+<wire x1="335.28" y1="53.34" x2="350.52" y2="53.34" width="0.1524" layer="91"/>
+<wire x1="350.52" y1="53.34" x2="350.52" y2="58.42" width="0.1524" layer="91"/>
+<pinref part="R18" gate="G$1" pin="2"/>
+<junction x="350.52" y="76.2"/>
 </segment>
 </net>
@@
 <wire x1="332.74" y1="35.56" x2="302.26" y2="35.56" width="0.1524" layer="91"/>
 <pinref part="R14" gate="G$1" pin="2"/>
-<wire x1="325.12" y1="30.48" x2="302.26" y2="30.48" width="0.1524" layer="91"/>
+<wire x1="317.5" y1="30.48" x2="302.26" y2="30.48" width="0.1524" layer="91"/>
 <junction x="302.26" y="30.48"/>
 <junction x="302.26" y="35.56"/>
@@
 <pinref part="R14" gate="G$1" pin="1"/>
 <pinref part="C25" gate="G$1" pin="P$2"/>
-<wire x1="335.28" y1="30.48" x2="340.36" y2="30.48" width="0.1524" layer="91"/>
+<wire x1="327.66" y1="30.48" x2="332.74" y2="30.48" width="0.1524" layer="91"/>
 </segment>
 </net>
@@
 <segment>
 <pinref part="C16" gate="G$1" pin="P$1"/>
-<wire x1="337.82" y1="35.56" x2="350.52" y2="35.56" width="0.1524" layer="91"/>
-<wire x1="350.52" y1="35.56" x2="350.52" y2="30.48" width="0.1524" layer="91"/>
+<wire x1="337.82" y1="35.56" x2="342.9" y2="35.56" width="0.1524" layer="91"/>
+<wire x1="342.9" y1="35.56" x2="342.9" y2="30.48" width="0.1524" layer="91"/>
 <pinref part="C25" gate="G$1" pin="P$1"/>
-<wire x1="350.52" y1="30.48" x2="345.44" y2="30.48" width="0.1524" layer="91"/>
+<wire x1="342.9" y1="30.48" x2="337.82" y2="30.48" width="0.1524" layer="91"/>
 <pinref part="R15" gate="G$1" pin="1"/>
+<wire x1="340.36" y1="12.7" x2="342.9" y2="12.7" width="0.1524" layer="91"/>
+<wire x1="342.9" y1="30.48" x2="342.9" y2="12.7" width="0.1524" layer="91"/>
+<junction x="342.9" y="30.48"/>
+<pinref part="R17" gate="G$1" pin="2"/>
+<wire x1="342.9" y1="12.7" x2="345.44" y2="12.7" width="0.1524" layer="91"/>
+</segment>
+</net>
+<net name="N$12" class="0">
+<segment>
 <pinref part="Q4" gate="G$1" pin="G"/>
-<wire x1="340.36" y1="12.7" x2="350.52" y2="12.7" width="0.1524" layer="91"/>
+<wire x1="358.14" y1="12.7" x2="363.22" y2="12.7" width="0.1524" layer="91"/>
 <pinref part="R16" gate="G$1" pin="1"/>
-<wire x1="350.52" y1="12.7" x2="358.14" y2="12.7" width="0.1524" layer="91"/>
-<wire x1="358.14" y1="12.7" x2="363.22" y2="12.7" width="0.1524" layer="91"/>
 <wire x1="358.14" y1="15.24" x2="358.14" y2="12.7" width="0.1524" layer="91"/>
-<wire x1="350.52" y1="30.48" x2="350.52" y2="12.7" width="0.1524" layer="91"/>
-<junction x="350.52" y="12.7"/>
-<junction x="358.14" y="12.7"/>
-<junction x="350.52" y="30.48"/>
-</segment>
-</net>
+<pinref part="R17" gate="G$1" pin="1"/>
+<wire x1="355.6" y1="12.7" x2="358.14" y2="12.7" width="0.1524" layer="91"/>
+</segment>
+</net>
+<net name="N$25" class="0">
+<segment>
+<pinref part="R11" gate="G$1" pin="1"/>
+<pinref part="Q3" gate="G$1" pin="G"/>
+<wire x1="365.76" y1="76.2" x2="360.68" y2="76.2" width="0.1524" layer="91"/>
+<wire x1="360.68" y1="76.2" x2="360.68" y2="71.12" width="0.1524" layer="91"/>
+<pinref part="R18" gate="G$1" pin="1"/>
+<junction x="360.68" y="76.2"/>
+</segment>
+</net>
